Commit message: add gripper

File: assets/xarm6/xarm6.urdf (robot description, URDF)
Before this commit: robot UF_ROBOT, 9 links, 8 joints
Links:
- added link left_finger, mass 0.048304; collision mesh filename=meshes/gripper/xarm/left_finger.stl; visual mesh filename=meshes/gripper/xarm/left_finger.stl
- added link left_inner_knuckle, mass 0.0230125781256706; collision mesh filename=meshes/gripper/xarm/left_inner_knuckle.stl; visual mesh filename=meshes/gripper/xarm/left_inner_knuckle.stl
- added link left_outer_knuckle, mass 0.033618; collision mesh filename=meshes/gripper/xarm/left_outer_knuckle.stl; visual mesh filename=meshes/gripper/xarm/left_outer_knuckle.stl
- added link link_tcp
- added link right_finger, mass 0.048304; collision mesh filename=meshes/gripper/xarm/right_finger.stl; visual mesh filename=meshes/gripper/xarm/right_finger.stl
- added link right_inner_knuckle, mass 0.023013; collision mesh filename=meshes/gripper/xarm/right_inner_knuckle.stl; visual mesh filename=meshes/gripper/xarm/right_inner_knuckle.stl
- added link right_outer_knuckle, mass 0.033618; collision mesh filename=meshes/gripper/xarm/right_outer_knuckle.stl; visual mesh filename=meshes/gripper/xarm/right_outer_knuckle.stl
- added link xarm_gripper_base_link, mass 0.54156; collision mesh filename=meshes/gripper/xarm/base_link.stl; visual mesh filename=meshes/gripper/xarm/base_link.stl
- link link1: geometry collision mesh filename=meshes/xarm6/visual/link1.stl; visual mesh filename=meshes/xarm6/visual/link1.stl
- link link2: geometry collision mesh filename=meshes/xarm6/visual/link2.stl; visual mesh filename=meshes/xarm6/visual/link2.stl
- link link3: geometry collision mesh filename=meshes/xarm6/visual/link3.stl; visual mesh filename=meshes/xarm6/visual/link3.stl
- link link4: geometry collision mesh filename=meshes/xarm6/visual/link4.stl; visual mesh filename=meshes/xarm6/visual/link4.stl
- link link5: geometry collision mesh filename=meshes/xarm6/visual/link5.stl; visual mesh filename=meshes/xarm6/visual/link5.stl
- link link6: geometry collision mesh filename=meshes/end_tool/collision/end_tool.stl; visual mesh filename=meshes/xarm6/visual/link6.stl
- link link_base: geometry collision mesh filename=meshes/xarm6/visual/link_base.stl; visual mesh filename=meshes/xarm6/visual/link_base.stl
Joints:
- added joint drive_joint: type revolute, parent xarm_gripper_base_link, child left_outer_knuckle, origin xyz=0 0.035 0.059098 rpy=0 0 0, axis 1 0 0, limit lower=0 upper=0.85 effort=50 velocity=2
- added joint gripper_fix: type fixed, parent link_eef, child xarm_gripper_base_link, origin xyz=0 0 0 rpy=0 0 0
- added joint joint_tcp: type fixed, parent xarm_gripper_base_link, child link_tcp, origin xyz=0 0 0.172 rpy=0 0 0
- added joint left_finger_joint: type revolute, parent left_outer_knuckle, child left_finger, origin xyz=0 0.035465 0.042039 rpy=0 0 0, axis -1 0 0, limit lower=0 upper=0.85 effort=50 velocity=2, mimic joint=drive_joint multiplier=1 offset=0
- added joint left_inner_knuckle_joint: type revolute, parent xarm_gripper_base_link, child left_inner_knuckle, origin xyz=0 0.02 0.074098 rpy=0 0 0, axis 1 0 0, limit lower=0 upper=0.85 effort=50 velocity=2, mimic joint=drive_joint multiplier=1 offset=0
- added joint right_finger_joint: type revolute, parent right_outer_knuckle, child right_finger, origin xyz=0 -0.035465 0.042039 rpy=0 0 0, axis 1 0 0, limit lower=0 upper=0.85 effort=50 velocity=2, mimic joint=drive_joint multiplier=1 offset=0
- added joint right_inner_knuckle_joint: type revolute, parent xarm_gripper_base_link, child right_inner_knuckle, origin xyz=0 -0.02 0.074098 rpy=0 0 0, axis -1 0 0, limit lower=0 upper=0.85 effort=50 velocity=2, mimic joint=drive_joint multiplier=1 offset=0
- added joint right_outer_knuckle_joint: type revolute, parent xarm_gripper_base_link, child right_outer_knuckle, origin xyz=0 -0.035 0.059098 rpy=0 0 0, axis -1 0 0, limit lower=0 upper=0.85 effort=50 velocity=2, mimic joint=drive_joint multiplier=1 offset=0
